File: resources/KiCad/RFIDwriter/RFIDwriter.kicad_sch (KiCad schematic)
At the start: 2 parts

Commit message: KiCad V9.0.1
Connections:
- net at U3. (3V3): now also U4. (SDA)
- net at U4. (SDA): no longer U3. (TX_GPIO_1)
- new net: U3. (3V3), U4. (SDA) (x5)
- now unconnected: U4. (SDA), U4. (SDA), U4. (SDA), U4. (SDA), U4. (SDA)
Changed lines of the file:
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@@
 (kicad_sch
-	(version 20231120)
+	(version 20250114)
 	(generator "eeschema")
-	(generator_version "8.0")
+	(generator_version "9.0")
 	(paper "USLetter")
 	(title_block
 		(title "RFIDwriter")
-		(date "2025-04-24")
+		(date "2025-05-08")
 		(rev "Rev 0.9")
 		(company "https://github.com/Mark-MDO47")
 	)
+	(text "Red"
+		(exclude_from_sim no)
+		(at 230.632 136.652 0)
+		(effects
+			(font
+				(size 1.5 1.5)
+			)
+		)
+	)
+	(text "Black"
+		(exclude_from_sim no)
+		(at 134.62 74.93 0)
+		(effects
+			(font
+				(size 1.5 1.5)
+			)
+		)
+	)
+	(text "Blue"
+		(exclude_from_sim no)
+		(at 134.62 80.264 0)
+		(effects
+			(font
+				(size 1.5 1.5)
+			)
+		)
+	)
+	(text "Blue"
+		(exclude_from_sim no)
+		(at 171.704 102.616 0)
+		(effects
+			(font
+				(size 1.5 1.5)
+			)
+		)
+	)
+	(text "Red"
+		(exclude_from_sim no)
+		(at 133.858 69.85 0)
+		(effects
+			(font
+				(size 1.5 1.5)
+			)
+		)
+	)
+	(text "Green\n"
+		(exclude_from_sim no)
+		(at 135.89 95.758 0)
+		(effects
+			(font
+				(size 1.5 1.5)
+			)
+		)
+	)
+	(text "Yellow"
+		(exclude_from_sim no)
+		(at 135.636 85.09 0)
+		(effects
+			(font
+				(size 1.5 1.5)
+			)
+		)
+	)
+	(text "White"
+		(exclude_from_sim no)
+		(at 135.636 90.424 0)
+		(effects
+			(font
+				(size 1.5 1.5)
+			)
+		)
+	)
+	(text "Yellow"
+		(exclude_from_sim no)
+		(at 168.91 125.476 0)
+		(effects
+			(font
+				(size 1.5 1.5)
+			)
+		)
+	)
+	(text "Black"
+		(exclude_from_sim no)
+		(at 169.164 129.54 0)
+		(effects
+			(font
+				(size 1.5 1.5)
+			)
+		)
+	)
+	(text "Green\n"
+		(exclude_from_sim no)
+		(at 171.45 94.742 0)
+		(effects
+			(font
+				(size 1.5 1.5)
+			)
+		)
+	)
+	(text "White"
+		(exclude_from_sim no)
+		(at 171.958 98.806 0)
+		(effects
+			(font
+				(size 1.5 1.5)
+			)
+		)
+	)
 	(wire
 		(pts
@@
 			(width 0)
 			(type default)
-		)
-	)
-	(text "Red"
-		(exclude_from_sim no)
-		(at 230.632 136.652 0)
-		(effects
-			(font
-				(size 1.5 1.5)
-			)
-		)
-	)
-	(text "Black"
-		(exclude_from_sim no)
-		(at 134.62 74.93 0)
-		(effects
-			(font
-				(size 1.5 1.5)
-			)
-		)
-	)
-	(text "Blue"
-		(exclude_from_sim no)
-		(at 134.62 80.264 0)
-		(effects
-			(font
-				(size 1.5 1.5)
-			)
-		)
-	)
-	(text "Blue"
-		(exclude_from_sim no)
-		(at 171.704 102.616 0)
-		(effects
-			(font
-				(size 1.5 1.5)
-			)
-		)
-	)
-	(text "Red"
-		(exclude_from_sim no)
-		(at 133.858 69.85 0)
-		(effects
-			(font
-				(size 1.5 1.5)
-			)
-		)
-	)
-	(text "Green\n"
-		(exclude_from_sim no)
-		(at 135.89 95.758 0)
-		(effects
-			(font
-				(size 1.5 1.5)
-			)
-		)
-	)
-	(text "Yellow"
-		(exclude_from_sim no)
-		(at 135.636 85.09 0)
-		(effects
-			(font
-				(size 1.5 1.5)
-			)
-		)
-	)
-	(text "White"
-		(exclude_from_sim no)
-		(at 135.636 90.424 0)
-		(effects
-			(font
-				(size 1.5 1.5)
-			)
-		)
-	)
-	(text "Yellow"
-		(exclude_from_sim no)
-		(at 168.91 125.476 0)
-		(effects
-			(font
-				(size 1.5 1.5)
-			)
-		)
-	)
-	(text "Black"
-		(exclude_from_sim no)
-		(at 169.164 129.54 0)
-		(effects
-			(font
-				(size 1.5 1.5)
-			)
-		)
-	)
-	(text "Green\n"
-		(exclude_from_sim no)
-		(at 171.45 94.742 0)
-		(effects
-			(font
-				(size 1.5 1.5)
-			)
-		)
-	)
-	(text "White"
-		(exclude_from_sim no)
-		(at 171.958 98.806 0)
-		(effects
-			(font
-				(size 1.5 1.5)
-			)
 		)
 	)
@@
 		)
 	)
+	(embedded_fonts no)
 )
