File: resources/KiCad/UniRemoteCYD/Battery_Power.kicad_sch (KiCad schematic)
At the start: 8 parts, among them J1 JST SM M 1x4, J2 JST SM F 1x4, J4 JST SM M 1x4, J5 ??? 1x2, J6 ??? 1x2, SW1 SW_SPST

Commit message: KiCad V9.0.1
Connections:
- net at SW1.~ (B): now also J1.2 (Pin_2)

Commit message: TOC
Connections:
- net at SW1.~ (B): now also J1.2 (Pin_2)
Other:
- note added: "JST SM 2 mm"
Changed lines of the file:
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@@
 	(generator "eeschema")
 	(generator_version "9.0")
-	(paper "A4")
+	(paper "USLetter")
 	(title_block
 		(title "UniRemoteCYD")
-		(date "2025-05-08")
-		(rev "Rev 0.9")
+		(date "2025-08-08")
+		(rev "Rev 1.0")
 		(company "https://github.com/Mark-MDO47")
 	)
@@
 		)
 	)
+	(text "JST SM\n2 mm"
+		(exclude_from_sim no)
+		(at 93.472 57.658 0)
+		(effects
+			(font
+				(size 2 2)
+			)
+		)
+	)
+	(text "JST SM\n2 mm"
+		(exclude_from_sim no)
+		(at 99.822 104.14 0)
+		(effects
+			(font
+				(size 2 2)
+			)
+		)
+	)
