File: resources/KiCad/UniRemoteCYD/UniRemoteCYD.kicad_sch (KiCad schematic)
At the start: 4 parts, among them J7 P1 F 1x4, J8 P1 M 1x4

Commit message: KiCad V9.0.1
Connections:
- net at U1. (DAT1): no longer U2. (SDA)
- new net: U1. (DAT1), U2. (MISO) (x5)
- now unconnected: U1. (VCC), U1. (VCC), U1. (VCC), U1. (VCC)
Changed lines of the file:
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@@
 (kicad_sch
-	(version 20231120)
+	(version 20250114)
 	(generator "eeschema")
-	(generator_version "8.0")
+	(generator_version "9.0")
 	(paper "USLetter")
 	(title_block
 		(title "UniRemoteCYD")
-		(date "2025-04-04")
+		(date "2025-05-08")
 		(rev "Rev 0.9")
 		(company "https://github.com/Mark-MDO47")
-	)
-	(wire
-		(pts
-			(xy 156.21 44.45) (xy 231.14 44.45)
-		)
-		(stroke
-			(width 0)
-			(type default)
-		)
-	)
-	(wire
-		(pts
-			(xy 156.21 57.15) (xy 231.14 57.15)
-		)
-		(stroke
-			(width 0)
-			(type default)
-		)
-	)
-	(wire
-		(pts
-			(xy 156.21 49.53) (xy 231.14 49.53)
-		)
-		(stroke
-			(width 0)
-			(type default)
-		)
-	)
-	(wire
-		(pts
-			(xy 156.21 54.61) (xy 231.14 54.61)
-		)
-		(stroke
-			(width 0)
-			(type default)
-		)
-	)
-	(wire
-		(pts
-			(xy 43.18 106.68) (xy 67.31 106.68)
-		)
-		(stroke
-			(width 0)
-			(type default)
-		)
-	)
-	(wire
-		(pts
-			(xy 156.21 52.07) (xy 231.14 52.07)
-		)
-		(stroke
-			(width 0)
-			(type default)
-		)
-	)
-	(wire
-		(pts
-			(xy 156.21 46.99) (xy 231.14 46.99)
-		)
-		(stroke
-			(width 0)
-			(type default)
-		)
-	)
-	(wire
-		(pts
-			(xy 43.18 114.3) (xy 67.31 114.3)
-		)
-		(stroke
-			(width 0)
-			(type default)
-		)
 	)
 	(rectangle
@@
 		)
 	)
+	(wire
+		(pts
+			(xy 156.21 44.45) (xy 231.14 44.45)
+		)
+		(stroke
+			(width 0)
+			(type default)
+		)
+	)
+	(wire
+		(pts
+			(xy 156.21 57.15) (xy 231.14 57.15)
+		)
+		(stroke
+			(width 0)
+			(type default)
+		)
+	)
+	(wire
+		(pts
+			(xy 156.21 49.53) (xy 231.14 49.53)
+		)
+		(stroke
+			(width 0)
+			(type default)
+		)
+	)
+	(wire
+		(pts
+			(xy 156.21 54.61) (xy 231.14 54.61)
+		)
+		(stroke
+			(width 0)
+			(type default)
+		)
+	)
+	(wire
+		(pts
+			(xy 43.18 106.68) (xy 67.31 106.68)
+		)
+		(stroke
+			(width 0)
+			(type default)
+		)
+	)
+	(wire
+		(pts
+			(xy 156.21 52.07) (xy 231.14 52.07)
+		)
+		(stroke
+			(width 0)
+			(type default)
+		)
+	)
+	(wire
+		(pts
+			(xy 156.21 46.99) (xy 231.14 46.99)
+		)
+		(stroke
+			(width 0)
+			(type default)
+		)
+	)
+	(wire
+		(pts
+			(xy 43.18 114.3) (xy 67.31 114.3)
+		)
+		(stroke
+			(width 0)
+			(type default)
+		)
+	)
 	(hierarchical_label "+5V "
 		(shape input)
 		(at 43.18 106.68 180)
-		(fields_autoplaced yes)
 		(effects
 			(font
@@
 		(shape input)
 		(at 43.18 114.3 180)
-		(fields_autoplaced yes)
 		(effects
 			(font
@@
 		(at 27.94 101.6)
 		(size 12.7 17.78)
+		(exclude_from_sim no)
+		(in_bom yes)
+		(on_board yes)
+		(dnp no)
 		(fields_autoplaced yes)
 		(stroke
@@
 		)
 	)
+	(embedded_fonts no)
 )

Commit message: TOC
Connections:
- net at U1. (DAT1): no longer U2. (MISO)
- new net: U1. (DAT1), U2. (MISO) (x5)
- now unconnected: U1. (DAT1), U1. (DAT1), U1. (DAT1), U1. (DAT1)
Other:
- note added: "JST MX 1.25 mm"
Changed lines of the file:
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@@
+		)
+	)
+	(text "JST MX\n1.25 mm"
+		(exclude_from_sim no)
+		(at 73.914 125.984 0)
+		(effects
+			(font
+				(size 2 2)
+			)
 		)
 	)

Commit message: update schematic with connector type/details
Connections:
- net at U1. (DAT1): no longer U2. (MISO)
- new net: U1. (DAT1), U2. (MISO) (x5)
- now unconnected: U1. (DAT1), U1. (DAT1), U1. (DAT1), U1. (DAT1)
Changed lines of the file:
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@@
 	(title_block
 		(title "UniRemoteCYD")
-		(date "2025-05-08")
-		(rev "Rev 0.9")
+		(date "2025-08-08")
+		(rev "Rev 1.0")
 		(company "https://github.com/Mark-MDO47")
 	)
